Commit message: odom being published

File: bot_description/urdf/bot.urdf.xacro (robot description, xacro)
@@ -9,9 +9,4 @@
     </inertial>
   </link>
-  <link name="base_footprint"/>
-  <joint name="base_ft_joint" type="fixed">
-    <parent link="base_link"/>
-    <child link="base_footprint"/>
-  </joint>
   <joint name="base_joint" type="fixed">
     <parent link="base_link"/>
@@ -302,4 +297,10 @@
         <odom_publish_frequency>50</odom_publish_frequency>
         <topic>/cmd_vel</topic>
+        <publish_odom>true</publish_odom>
+        <publish_odom_tf>true</publish_odom_tf>
+        <publish_wheel_tf>true</publish_wheel_tf>
+        <odom_topic>odom</odom_topic>
+        <frame_id>odom</frame_id>
+        <child_frame_id>base_link</child_frame_id>
       </plugin>
     </gazebo>

Commit message: diff drive controller config

File: bot_description/urdf/bot.urdf.xacro (robot description, xacro)
@@ -2,4 +2,11 @@
   <robot name="bot" xmlns:xacro="http://ros.org/wiki/xacro">
   <xacro:include filename="bot_ros2_control.xacro" />
+    <joint name="base_footprint_joint" type="fixed">
+        <parent link="base_link"/>
+        <child link="base_footprint"/>
+        <origin xyz="0 0 0" rpy="0 0 0"/>
+    </joint>
+    <link name="base_footprint">
+    </link>
   <link name="base_link">
       <inertial>
@@ -282,5 +289,5 @@
     <gazebo>
         <plugin filename="ign_ros2_control-system" name="ign_ros2_control::IgnitionROS2ControlPlugin">
-          <parameters></parameters>
+          <parameters>$(find bot_controller)/config/bot_controller.yaml</parameters>
         </plugin>
         <plugin filename="ignition-gazebo-imu-system" name="ignition::gazebo::systems::Imu"></plugin>
@@ -288,5 +295,5 @@
         <render_engine>ogre2</render_engine>
       </plugin>
-      <plugin filename="ignition-gazebo-diff-drive-system"
+<!--      <plugin filename="ignition-gazebo-diff-drive-system"
         name="ignition::gazebo::systems::DiffDrive">
         <left_joint>wheel_front_left_joint</left_joint>
@@ -298,5 +305,4 @@
         <odom_publish_frequency>50</odom_publish_frequency>
         <topic>/cmd_vel</topic>
-    <!-- Make sure you have these exact parameters -->
         <publish_odom>true</publish_odom>
         <publish_odom_tf>true</publish_odom_tf>
@@ -304,7 +310,7 @@
         <frame_id>odom</frame_id>
         <child_frame_id>base_link</child_frame_id>
-        <!-- Add this parameter -->
         <tf_topic>tf</tf_topic>
       </plugin>
+       -->
     </gazebo>
 </robot>

Commit message: odom fixed

File: bot_description/urdf/bot.urdf.xacro (robot description, xacro)
@@ -2,12 +2,5 @@
   <robot name="bot" xmlns:xacro="http://ros.org/wiki/xacro">
   <xacro:include filename="bot_ros2_control.xacro" />
-    <joint name="base_footprint_joint" type="fixed">
-        <parent link="base_link"/>
-        <child link="base_footprint"/>
-        <origin xyz="0 0 0" rpy="0 0 0"/>
-    </joint>
-    <link name="base_footprint">
-    </link>
-  <link name="base_link">
+  <link name="base_footprint">
       <inertial>
             <mass value="2" />
@@ -17,9 +10,9 @@
   </link>
   <joint name="base_joint" type="fixed">
-    <parent link="base_link"/>
-    <child link="chassis"/>
+    <parent link="base_footprint"/>
+    <child link="base_link"/>
     <origin xyz="0.0 0.0 0.15" rpy="0.0 0.0 0.0"/>
   </joint>
-  <link name="chassis">
+  <link name="base_link">
     <visual>
       <geometry>
@@ -63,5 +56,5 @@
   <joint name="wheel_front_right_joint" type="continuous">
     <origin xyz="0.25 0.4 -0.05" rpy="1.57 0.0 0.0"/>
-    <parent link="chassis"/>
+    <parent link="base_link"/>
     <child link="wheel_front_right"/>
     <axis xyz="0.0 0.0 1.0"/>
@@ -89,5 +82,5 @@
   <joint name="wheel_front_left_joint" type="continuous">
     <origin xyz="0.25 -0.4 -0.05" rpy="1.57 0.0 0.0"/>
-    <parent link="chassis"/>
+    <parent link="base_link"/>
     <child link="wheel_front_left"/>
     <axis xyz="0.0 0.0 1.0"/>
@@ -115,5 +108,5 @@
   <joint name="wheel_back_right_joint" type="continuous">
     <origin xyz="-0.25 0.4 -0.05" rpy="1.57 0.0 0.0"/>
-    <parent link="chassis"/>
+    <parent link="base_link"/>
     <child link="wheel_back_right"/>
     <axis xyz="0.0 0.0 1.0"/>
@@ -141,5 +134,5 @@
   <joint name="wheel_back_left_joint" type="continuous">
     <origin xyz="-0.25 -0.4 -0.05" rpy="1.57 0.0 0.0"/>
-    <parent link="chassis"/>
+    <parent link="base_link"/>
     <child link="wheel_back_left"/>
     <axis xyz="0.0 0.0 1.0"/>
@@ -167,5 +160,5 @@
   <joint name="camera_joint" type="fixed">
     <origin xyz="-0.43 0 0.0" rpy="0 0.0 3.14"/>
-    <parent link="chassis"/>
+    <parent link="base_link"/>
     <child link="rgb_camera"/>
     <axis xyz="0.0 0 0"/>
@@ -218,5 +211,5 @@
   <joint name="laser_joint" type="fixed">
     <origin xyz="0 0 0.15" rpy="0 0.0 3.14"/>
-    <parent link="chassis"/>
+    <parent link="base_link"/>
     <child link="laser_link"/>
     <axis xyz="0.0 0.0 1.0"/>
@@ -295,22 +288,4 @@
         <render_engine>ogre2</render_engine>
       </plugin>
-<!--      <plugin filename="ignition-gazebo-diff-drive-system"
-        name="ignition::gazebo::systems::DiffDrive">
-        <left_joint>wheel_front_left_joint</left_joint>
-        <left_joint>wheel_back_left_joint</left_joint>
-        <right_joint>wheel_front_right_joint</right_joint>
-        <right_joint>wheel_back_right_joint</right_joint>
-        <wheel_separation>0.8</wheel_separation>
-        <wheel_radius>0.1</wheel_radius>
-        <odom_publish_frequency>50</odom_publish_frequency>
-        <topic>/cmd_vel</topic>
-        <publish_odom>true</publish_odom>
-        <publish_odom_tf>true</publish_odom_tf>
-        <odom_topic>odom</odom_topic>
-        <frame_id>odom</frame_id>
-        <child_frame_id>base_link</child_frame_id>
-        <tf_topic>tf</tf_topic>
-      </plugin>
-       -->
     </gazebo>
 </robot>

Commit message: odom drift partially fixed

File: bot_description/urdf/bot.urdf.xacro (robot description, xacro)
@@ -12,5 +12,5 @@
     <parent link="base_footprint"/>
     <child link="base_link"/>
-    <origin xyz="0.0 0.0 0.15" rpy="0.0 0.0 0.0"/>
+    <origin xyz="0.0 0.0 0.15" rpy="0.0 0.0 3.14159"/>  <!-- Add 180-degree rotation -->
   </joint>
   <link name="base_link">
@@ -54,10 +54,4 @@
     </collision>
   </link>
-  <joint name="wheel_front_right_joint" type="continuous">
-    <origin xyz="0.25 0.4 -0.05" rpy="1.57 0.0 0.0"/>
-    <parent link="base_link"/>
-    <child link="wheel_front_right"/>
-    <axis xyz="0.0 0.0 1.0"/>
-  </joint>
   <link name="wheel_front_left">
     <inertial>
@@ -80,10 +74,4 @@
     </collision>
   </link>
-  <joint name="wheel_front_left_joint" type="continuous">
-    <origin xyz="0.25 -0.4 -0.05" rpy="1.57 0.0 0.0"/>
-    <parent link="base_link"/>
-    <child link="wheel_front_left"/>
-    <axis xyz="0.0 0.0 1.0"/>
-  </joint>
 <link name="wheel_back_right">
     <inertial>
@@ -106,10 +94,4 @@
     </collision>
   </link>
-  <joint name="wheel_back_right_joint" type="continuous">
-    <origin xyz="-0.25 0.4 -0.05" rpy="1.57 0.0 0.0"/>
-    <parent link="base_link"/>
-    <child link="wheel_back_right"/>
-    <axis xyz="0.0 0.0 1.0"/>
-  </joint>
   <link name="wheel_back_left">
     <inertial>
@@ -132,10 +114,4 @@
     </collision>
   </link>
-  <joint name="wheel_back_left_joint" type="continuous">
-    <origin xyz="-0.25 -0.4 -0.05" rpy="1.57 0.0 0.0"/>
-    <parent link="base_link"/>
-    <child link="wheel_back_left"/>
-    <axis xyz="0.0 0.0 1.0"/>
-  </joint>
   <link name="rgb_camera">
     <inertial>
@@ -244,39 +220,63 @@
     </sensor>
   </gazebo>
+    <joint name="wheel_front_right_joint" type="continuous">
+    <origin xyz="-0.25 0.4 -0.05" rpy="1.57 0.0 0.0"/>
+    <parent link="base_link"/>
+    <child link="wheel_front_right"/>
+    <axis xyz="0.0 0.0 1.0"/>
+  </joint>
+  <joint name="wheel_front_left_joint" type="continuous">
+    <origin xyz="-0.25 -0.4 -0.05" rpy="1.57 0.0 0.0"/>
+    <parent link="base_link"/>
+    <child link="wheel_front_left"/>
+    <axis xyz="0.0 0.0 1.0"/>
+  </joint>
+    <joint name="wheel_back_right_joint" type="continuous">
+    <origin xyz="0.25 0.4 -0.05" rpy="1.57 0.0 0.0"/>
+    <parent link="base_link"/>
+    <child link="wheel_back_right"/>
+    <axis xyz="0.0 0.0 1.0"/>
+  </joint>
+  <joint name="wheel_back_left_joint" type="continuous">
+    <origin xyz="0.25 -0.4 -0.05" rpy="1.57 0.0 0.0"/>
+    <parent link="base_link"/>
+    <child link="wheel_back_left"/>
+    <axis xyz="0.0 0.0 1.0"/>
+  </joint>
     <gazebo reference="wheel_front_right">
-      <mu1>1.0</mu1>
-      <mu2>1.0</mu2>
-      <kp>500000.0</kp>
-      <kd>10.0</kd>
-      <minDepth>0.001</minDepth>
-      <maxVel>1</maxVel>
-      <fdir1>1 0 0</fdir1>
+    <mu1>1000000000000000.0</mu1>
+    <mu2>1000000000000000.0</mu2>
+    <kp>1000000000000.0</kp>
+    <kd>10.0</kd>
+    <minDepth>0.001</minDepth>
+    <maxVel>0.1</maxVel>
+    <fdir1>1 0 0</fdir1>
     </gazebo>
     <gazebo reference="wheel_front_left">
-      <mu1>1.0</mu1>
-      <mu2>1.0</mu2>
-      <kp>500000.0</kp>
-      <kd>10.0</kd>
-      <minDepth>0.001</minDepth>
-      <maxVel>1</maxVel>
-      <fdir1>1 0 0</fdir1>
+    <mu1>1000000000000000.0</mu1>
+    <mu2>1000000000000000.0</mu2>
+    <kp>1000000000000.0</kp>
+    <kd>10.0</kd>
+    <minDepth>0.001</minDepth>
+    <maxVel>0.1</maxVel>
+    <fdir1>1 0 0</fdir1>
     </gazebo>
     <gazebo reference="wheel_back_right">
-      <mu1>1.0</mu1>
-      <mu2>1.0</mu2>
-      <kp>500000.0</kp>
-      <kd>10.0</kd>
-      <minDepth>0.001</minDepth>
-      <maxVel>1</maxVel>
-      <fdir1>1 0 0</fdir1>
+    <mu1>1000000000000000.0</mu1>
+    <mu2>1000000000000000.0</mu2>
+    <kp>1000000000000.0</kp>
+    <kd>10.0</kd>
+    <minDepth>0.001</minDepth>
+    <maxVel>0.1</maxVel>
+    <fdir1>1 0 0</fdir1>
     </gazebo>
     <gazebo reference="wheel_back_left">
-      <mu1>1.0</mu1>
-      <mu2>1.0</mu2>
-      <kp>500000.0</kp>
-      <kd>10.0</kd>
-      <minDepth>0.001</minDepth>
-      <maxVel>1</maxVel>
-      <fdir1>1 0 0</fdir1>
+    <mu1>1000000000000000.0</mu1>
+    <mu2>1000000000000000.0</mu2>
+    <kp>1000000000000.0</kp>
+    <kd>10.0</kd>
+    <minDepth>0.001</minDepth>
+    <maxVel>0.1</maxVel>
+    <fdir1>1 0 0</fdir1>
     </gazebo>
     <gazebo>

Commit message: SLAM working

File: bot_description/urdf/bot.urdf.xacro (robot description, xacro)
@@ -12,5 +12,5 @@
     <parent link="base_footprint"/>
     <child link="base_link"/>
-    <origin xyz="0.0 0.0 0.15" rpy="0.0 0.0 3.14159"/>  <!-- Add 180-degree rotation -->
+    <origin xyz="0.0 0.0 0.15" rpy="0.0 0.0 3.14159"/>
   </joint>
   <link name="base_link">
@@ -50,5 +50,5 @@
     <collision>
       <geometry>
-          <cylinder radius="0.10" length="0.1"/>
+          <sphere radius="0.10"/>
       </geometry>
     </collision>
@@ -70,5 +70,5 @@
     <collision>
       <geometry>
-          <cylinder radius="0.10" length="0.1"/>
+          <sphere radius="0.10" />
       </geometry>
     </collision>
@@ -90,5 +90,5 @@
     <collision>
       <geometry>
-          <cylinder radius="0.10" length="0.1"/>
+          <sphere radius="0.10" />
       </geometry>
     </collision>
@@ -110,5 +110,5 @@
     <collision>
       <geometry>
-          <cylinder radius="0.10" length="0.1"/>
+          <sphere radius="0.10"/>
       </geometry>
     </collision>

Commit message: added 3d lidar support

File: bot_description/urdf/bot.urdf.xacro (robot description, xacro)
@@ -191,5 +191,6 @@
     <axis xyz="0.0 0.0 1.0"/>
   </joint>
-  <gazebo reference="laser_link">
+    <!-- 2D LIDAR-->
+<!--  <gazebo reference="laser_link">
     <sensor name="lidar" type="gpu_lidar">
       <always_on>true</always_on>
@@ -219,4 +220,55 @@
       </lidar>
     </sensor>
+  </gazebo>-->
+  <!-- velodyne vlp-32 3D lidar plugin-->
+  <gazebo reference="laser_link">
+    <sensor name="lidar" type="gpu_lidar">
+      <update_rate>10</update_rate>
+      <topic>scan</topic>
+      <gz_frame_id>laser_link</gz_frame_id>
+      <lidar>
+        <scan>
+          <horizontal>
+            <samples>720</samples>
+            <resolution>1</resolution>
+            <min_angle>-3.14156</min_angle>
+            <max_angle>3.14156</max_angle>
+          </horizontal>
+          <vertical>
+            <samples>32</samples>
+            <min_angle>-0.5353</min_angle>
+            <max_angle>0.1862</max_angle>
+          </vertical>
+        </scan>
+        <range>
+          <min>0.05</min>
+          <max>10.0</max>
+          <resolution>0.01</resolution>
+        </range>
+        <noise>
+            <type>gaussian</type>
+            <mean>0.0</mean>
+            <stddev>0.01</stddev>
+        </noise>
+        <frame_id>scan_link</frame_id>
+      </lidar>
+      <always_on>1</always_on>
+      <visualize>true</visualize>
+    </sensor>
+  </gazebo>
+  <joint name="navsat_joint" type="fixed">
+    <origin xyz="0 0 0" rpy="0 0 0" />
+    <parent link="base_link"/>
+    <child link="navsat_link" />
+  </joint>
+  <link name="navsat_link">
+  </link>
+  <gazebo reference="navsat_link">
+    <sensor name="navsat" type="navsat">
+      <always_on>1</always_on>
+      <update_rate>1</update_rate>
+      <topic>navsat</topic>
+      <gz_frame_id>navsat_link</gz_frame_id>
+    </sensor>
   </gazebo>
     <joint name="wheel_front_right_joint" type="continuous">
@@ -288,4 +340,17 @@
         <render_engine>ogre2</render_engine>
       </plugin>
+        <plugin
+        filename="gz-sim-navsat-system"
+        name="gz::sim::systems::NavSat">
+      </plugin>
+      <!-- Set the coordinates for the world origin -->
+      <spherical_coordinates>
+        <surface_model>EARTH_WGS84</surface_model>
+        <world_frame_orientation>ENU</world_frame_orientation>
+        <latitude_deg>47.478950</latitude_deg>
+        <longitude_deg>19.057785</longitude_deg>
+        <elevation>0</elevation>
+        <heading_deg>0</heading_deg>
+      </spherical_coordinates>
     </gazebo>
 </robot>
